File: pcb/pas_chiffre.kicad_pcb (KiCad board)
At the start: 2 copper layers, 96.3 x 89 mm, 26 parts, among them J1 Conn_01x06_Pin, J2 Conn_01x06_Pin, SW1 SW_SPST, SW10 SW_SPST, SW11 SW_SPST, SW12 SW_SPST, SW13 SW_SPST, SW14 SW_SPST, SW15 SW_SPST, SW16 SW_SPST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

Commit message: reshuffling
Other:
- board size 96.3 x 89 mm -> 96.3 x 87.5 mm
