File: pcb/pas_chiffre.kicad_sch (KiCad schematic)
At the start: 26 parts, among them J1 Conn_01x06_Pin, J2 Conn_01x06_Pin, SW1 SW_SPST, SW10 SW_SPST, SW11 SW_SPST, SW12 SW_SPST, SW13 SW_SPST, SW14 SW_SPST, SW15 SW_SPST, SW16 SW_SPST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

Commit message: fixed switch footprint
Parts:
- SW1, SW10, SW11, SW12, SW13, SW14, SW15, SW16, SW17, SW2, SW3, SW4, SW5, SW6, SW7, SW8, SW9: footprint keyswitches:SW_MX_reversible_minimal -> keyswitches:SW_MX_reversible
